Commit message: modify robot model

File: urdf/my_robot.xacro (robot description, xacro)
@@ -129,5 +129,5 @@
     <parent link="base_link"/>
     <child link="right_wheel"/>
-    <origin xyz="0 0.2 -0.25"/>
+    <origin xyz="0 -0.2 -0.25"/>
     <axis xyz="0 1 0" rpy="0 0 0"/>
     <limit effort="10000" velocity="1000"/>
@@ -163,5 +163,5 @@
     <parent link="base_link"/>
     <child link="left_wheel"/>
-    <origin xyz="0 -0.2 -0.25"/>
+    <origin xyz="0 0.2 -0.25"/>
     <axis xyz="0 1 0" rpy="0 0 0"/>
     <limit effort="10000" velocity="1000"/>

Commit message: rtabmap

File: urdf/my_robot.xacro (robot description, xacro)
@@ -102,4 +102,11 @@
     <origin xyz="0.1814 0 0.1414"/>
   </joint>
+  <joint name="camera_optical_joint" type="fixed">
+    <origin xyz="0 0 0" rpy="-1.5707 0 -1.5707"/>
+    <parent link="camera"/>
+    <child link="camera_link_optical"/>
+  </joint>
+  <link name="camera_link_optical">
+  </link>
   <link name="right_wheel">
     <inertial>
